File: EmilyProgress/IntroNewPiHat/IntroNewPiHat.kicad_sch (KiCad schematic)
At the start: 18 parts, among them J1 RPi_GPIO, J2 Conn_01x03_Pin, J3 Conn_01x03_Pin, J4 Conn_01x04_Pin

Commit message: update 12/1/2024
Parts:
- removed IMU1: HEADER-1X476MIL, Adafruit BNO055:1X04_ROUND_76, symbol RPi_Hat_V2-eagle-import:HEADER-1X476MIL
- removed IMU2: HEADER-1X6, Adafruit BNO055:Adafruit_BPO055, symbol Adafruit BNO055-eagle-import:HEADER-1X6
- removed J?: Conn_01x02_Pin, symbol Connector:Conn_01x02_Pin
- removed J?: Conn_01x03_Pin, Connector_PinHeader_2.54mm:PinHeader_1x03_P2.54mm_Horizontal, symbol Connector:Conn_01x03_Pin
- added IMU_HEADER1: HEADER-1X6, Adafruit BNO055:Adafruit_BPO055, symbol Adafruit_library:HEADER-1X6
- added J10: Conn_01x03_Pin, Connector_PinHeader_2.54mm:PinHeader_1x03_P2.54mm_Horizontal, symbol Connector:Conn_01x03_Pin
- added J8: XT30PW-M, XT30PW-M:AMASS_XT30PW-M, symbol XT30PW-M:XT30PW-M
- added JP1: HEADER-1X476MIL, Adafruit BNO055:1X04_ROUND_76, symbol RPi_Hat_V2-eagle-import:HEADER-1X476MIL
- J16: renamed from J3; footprint Connector_PinHeader_2.54mm:PinHeader_1x03_P2.54mm_Vertical -> Connector_PinHeader_2.54mm:PinHeader_1x03_P2.54mm_Horizontal
- J7: renamed from J1; footprint Samtec_HLE-120-02-XXX-DV-BE-XX-XX:Samtec_HLE-120-02-XXX-DV-BE-XX-XX -> RPi_HatSamtec_HLE-120-02-XXX-DV-BE-XX-XX:Samtec_HLE-120-02-XXX-DV-BE-XX-XX
- gave numbers to parts that had none: 10
- renumbered J4 to J2, J2 to J5
Connections:
- net GND: now also IMU_HEADER1.B3 (3_(GND)), J10.1 (Pin_1), J8.N
- net PWM0: now also J5.1 (Pin_1); no longer J16.3 (Pin_3)
- net PWM1: no longer J5.1 (Pin_1)
- net PWM3: now also J4.3 (Pin_3)
- net PWR: now also IMU_HEADER1.B1, J8.P, JP1.3
- net RST: now also IMU_HEADER1.B6
- net RX10: now also IMU_HEADER1.B4 (4)
- net S221: now also J10.3 (Pin_3)
- net TX08: now also IMU_HEADER1.B5 (5)
- net PIN17: now reaches J7.11 (BCM17)
- net PIN17: now also J16.3 (Pin_3)
- no-connect marks 5 -> 31
Other:
- moved on the sheet: J11, J12, J13, J14, J15, J16, J9
